Commit message: Set rotor_drag_coefficient and rolling_moment_coefficient to 0 as they are not modelled.

File: rotors_description/urdf/hummingbird.xacro (robot description, xacro)
@@ -35,6 +35,6 @@
   <xacro:property name="time_constant_down" value="0.025" /> <!-- [s] -->
   <xacro:property name="max_rot_velocity" value="838" /> <!-- [rad/s] -->
-  <xacro:property name="rotor_drag_coefficient" value="8.06428e-05" />
-  <xacro:property name="rolling_moment_coefficient" value="0.000001" />
+  <xacro:property name="rotor_drag_coefficient" value="0.0" />
+  <xacro:property name="rolling_moment_coefficient" value="0.0" />
   <!-- Property Blocks -->
   <xacro:property name="body_inertia">
